File: schematics/fpga_io_b.kicad_sch (KiCad schematic)
At the start: 12 parts, among them J2 2.54mm Through-Hole Socket, J3 2.54mm Through-Hole Socket, U1B XC7AxxT-xCSG325, U1C XC7AxxT-xCSG325, U1D XC7AxxT-xCSG325, U2 S25Q

Commit message: finished schematics
Connections:
- net DIO_3_N: now also J2.24 (Pin_24); no longer J2.25 (Pin_25)
- net DIO_3_P: now also J2.25 (Pin_25); no longer J2.24 (Pin_24)
- net DIO_5_N: now also J2.18 (Pin_18)
- net DIO_5_P: now also J2.19 (Pin_19)
- net DIO_6_N: now also J3.22 (Pin_22)
- net DIO_6_P: now also J3.21 (Pin_21)
- net DIO_7_N: now also J2.15 (Pin_15)
- net DIO_7_P: now also J2.16 (Pin_16)
- net XADC_2_N: now also J2.30 (Pin_30); no longer J2.31 (Pin_31)
- net XADC_2_P: now also J2.31 (Pin_31); no longer J2.30 (Pin_30)
- net XADC_3_N: now also J2.27 (Pin_27); no longer J2.28 (Pin_28)
- net XADC_3_P: now also J2.28 (Pin_28); no longer J2.27 (Pin_27)
- net DIO_9_N: now reaches U1D.J4 (IO_L2N_T0_34)
- net DIO_9_N: now also J2.12 (Pin_12)
- net DIO_9_P: now reaches U1D.J5 (IO_L2P_T0_34)
- net DIO_9_P: now also J2.13 (Pin_13)
- net DIO_10_P: now reaches U1D.K3 (IO_L4P_T0_34)
- net DIO_10_P: now also J3.27 (Pin_27)
- net DIO_8_N: now reaches U1D.K5 (IO_L1N_T0_34)
- net DIO_8_N: now also J3.25 (Pin_25)
- net DIO_8_P: now reaches U1D.K6 (IO_L1P_T0_34)
- net DIO_8_P: now also J3.24 (Pin_24)
- net DIO_10_N: now reaches U1D.L2 (IO_L4N_T0_34)
- net DIO_10_N: now also J3.28 (Pin_28)
- net DIO_11_N: now reaches U1D.L3 (IO_L5N_T0_34)
- net DIO_11_N: now also J2.9 (Pin_9)
- net DIO_11_P: now reaches U1D.L4 (IO_L5P_T0_34)
- net DIO_11_P: now also J2.10 (Pin_10)
- net DIO_12_N: now reaches U1D.M1 (IO_L7N_T1_34)
- net DIO_12_N: now also J3.31 (Pin_31)
- net DIO_12_P: now reaches U1D.M2 (IO_L7P_T1_34)
- net DIO_12_P: now also J3.30 (Pin_30)
- net DIO_14_P: now reaches U1D.M4 (IO_L10P_T1_34)
- net DIO_14_P: now also J3.33 (Pin_33)
- net DIO_13_P: now reaches U1D.M6 (IO_L8P_T1_34)
- net DIO_13_P: now also J2.7 (Pin_7)
- net DIO_14_N: now reaches U1D.N4 (IO_L10N_T1_34)
- net DIO_14_N: now also J3.34 (Pin_34)
- net DIO_13_N: now reaches U1D.N6 (IO_L8N_T1_34)
- net DIO_13_N: now also J2.6 (Pin_6)
- net DIO_15_N: now reaches U1D.T3 (IO_L17N_T2_34)
- net DIO_15_N: now also J2.3 (Pin_3)
- net DIO_15_P: now reaches U1D.T4 (IO_L17P_T2_34)
- net DIO_15_P: now also J2.4 (Pin_4)
- net DIO_16_P: now reaches U1D.U4 (IO_L18P_T2_34)
- net DIO_16_P: now also J3.36 (Pin_36)
- net DIO_16_N: now reaches U1D.V4 (IO_L18N_T2_34)
- net DIO_16_N: now also J3.37 (Pin_37)
- no-connect marks 94 -> 90
