File: designs/schematics/M2_edge_b.kicad_sch (KiCad schematic)
At the start: 11 parts, among them J1 Bus_PCI_Express_x4, P2 USB_C_Plug_USB2.0

Commit message: Add files via upload
Parts:
- P2: footprint (none) -> Connector_USB:USB_C_Plug_JAE_DX07P024AJ1
- R_CC_PD1: renamed from R_CC_PD; footprint (none) -> Resistor_SMD:R_0201_0603Metric
Connections:
- no-connect marks 24 -> 28
Changed lines of the file:
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@@
+	)
+	(no_connect
+		(at 185.42 77.47)
 	)
 	(no_connect
@@
 	)
 	(no_connect
+		(at 154.94 77.47)
+	)
+	(no_connect
 		(at 185.42 31.75)
+	)
+	(no_connect
+		(at 185.42 80.01)
 	)
 	(no_connect
@@
 	)
 	(no_connect
+		(at 154.94 80.01)
+	)
+	(no_connect
 		(at 185.42 36.83)
 	)
@@
 	)
 	(global_label "MGT1_TX_B+"
-		(shape input)
+		(shape output)
 		(at 123.19 72.39 180)
 		(effects
@@
 	)
 	(global_label "MGT0_TX_B-"
-		(shape input)
+		(shape output)
 		(at 123.19 69.85 180)
 		(effects
@@
 	)
 	(global_label "MGT_REFCLK0_B+"
-		(shape input)
+		(shape output)
 		(at 128.27 44.45 180)
 		(effects
@@
 	)
 	(global_label "MGT0_TX_B+"
-		(shape input)
+		(shape output)
 		(at 123.19 67.31 180)
 		(effects
@@
 	)
 	(global_label "MGT_REFCLK0_B-"
-		(shape input)
+		(shape output)
 		(at 128.27 46.99 180)
 		(effects
@@
 	)
 	(global_label "MGT1_TX_B-"
-		(shape input)
+		(shape output)
 		(at 123.19 74.93 180)
 		(effects
@@
 		(dnp no)
 		(fields_autoplaced yes)
-		(property "Reference" "R_CC_PD"
+		(property "Reference" "R_CC_PD1"
 			(at 78.74 127 90)
 			(effects
@@
 			)
 		)
-		(property "Footprint" ""
+		(property "Footprint" "Resistor_SMD:R_0201_0603Metric"
 			(at 78.74 135.128 90)
 			(effects
@@
 			(project ""
 				(path "/425a64d6-34ec-416c-8211-1f7c9aeb5428/00000000-0000-0000-0000-0000588189a7"
-					(reference "R_CC_PD")
+					(reference "R_CC_PD1")
 					(unit 1)
 				)
@@
 			)
 		)
-		(property "Footprint" ""
+		(property "Footprint" "Connector_USB:USB_C_Plug_JAE_DX07P024AJ1"
 			(at 62.23 143.51 0)
 			(effects
