File: designs/schematics/USB_IO_b.kicad_sch (KiCad schematic)
At the start: 4 parts, among them U7 FT230XQ

Commit message: Add files via upload
Parts:
- U7: footprint Housings_DFN_QFN:QFN-16-1EP_4x4mm_Pitch0.65mm -> fp_archive:QFN65P400X400X80-17N
Changed lines of the file:
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@@
 			)
 		)
-		(property "Footprint" "Housings_DFN_QFN:QFN-16-1EP_4x4mm_Pitch0.65mm"
+		(property "Footprint" "fp_archive:QFN65P400X400X80-17N"
 			(at 116.84 60.96 0)
 			(effects
