File: designs/schematics/fpga_io_b.kicad_sch (KiCad schematic)
At the start: 10 parts, among them U1B XC7AxxT-xCSG325, U1C XC7AxxT-xCSG325, U1D XC7AxxT-xCSG325, U2 S25Q

Commit message: Add files via upload
Parts:
- D2, D3, D4: footprint LEDs:LED_0402 -> fp_archive:LED_0402
- RN2, RN3: footprint Resistors_SMD:R_Array_Convex_4x0402 -> Resistor_SMD:R_Array_Convex_4x0402
- U2: footprint Housings_SOIC:SOIC-8_3.9x4.9mm_Pitch1.27mm -> fp_archive:SOIC-8_3.9x4.9mm_Pitch1.27mm
- renumbered U1B to U1B1, U1C to U1C1, U1D to U1D1
