File: designs/schematics/fpga_pcie_b.kicad_sch (KiCad schematic)
At the start: 2 parts, among them U1E XC7AxxT-xCSG325

Commit message: Add files via upload
Parts:
- renumbered U1E to U1E1
Changed lines of the file:
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@@
 	)
 	(global_label "MGT0_RX_B+"
-		(shape input)
+		(shape output)
 		(at 111.76 82.55 180)
 		(effects
@@
 	)
 	(global_label "MGT0_RX_B-"
-		(shape input)
+		(shape output)
 		(at 111.76 85.09 180)
 		(effects
@@
 	)
 	(global_label "P1V2_MGTAVTT_B"
-		(shape input)
+		(shape output)
 		(at 101.6 48.26 180)
 		(effects
@@
 	)
 	(global_label "MGT1_RX_B-"
-		(shape input)
+		(shape output)
 		(at 80.01 69.85 180)
 		(effects
@@
 	)
 	(global_label "MGT1_RX_B+"
-		(shape input)
+		(shape output)
 		(at 80.01 67.31 180)
 		(effects
@@
 		(on_board yes)
 		(dnp no)
-		(property "Reference" "U1E"
+		(property "Reference" "U1E1"
 			(at 120.65 45.72 0)
 			(effects
@@
 			(project "PicoEVB"
 				(path "/425a64d6-34ec-416c-8211-1f7c9aeb5428/00000000-0000-0000-0000-0000594f3239"
-					(reference "U1E")
+					(reference "U1E1")
 					(unit 5)
 				)
