File: designs/schematics/fpga_pwr_cfg_b.kicad_sch (KiCad schematic)
At the start: 54 parts, among them U1A XC7AxxT-xCSG325, U1F XC7AxxT-xCSG325

Commit message: Add files via upload
Parts:
- C27, C28, C29, C30, C4: footprint Capacitors_SMD:C_0603 -> fp_archive:C_0603
- C3: footprint Capacitors_SMD:C_0805 -> fp_archive:C_0805
- D1: footprint LEDs:LED_0402 -> fp_archive:LED_0402
- RN1: footprint Resistors_SMD:R_Array_Convex_4x0402 -> Resistor_SMD:R_Array_Convex_4x0402
- U1A1: renamed from U1A; footprint (none) -> XC7A50T-CSG325:CSG-324
- renumbered U1F to U1F1
Changed lines of the file:
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@@
 	)
 	(global_label "VCC_BANK15_B"
-		(shape output)
+		(shape input)
 		(at 203.2 68.58 0)
 		(effects
@@
 	)
 	(global_label "FPGA_CCLK_0_B"
-		(shape output)
+		(shape input)
 		(at 80.01 152.4 180)
 		(effects
@@
 	)
 	(global_label "VCC_BANK14_B"
-		(shape output)
+		(shape input)
 		(at 203.2 57.15 0)
 		(effects
@@
 	)
 	(global_label "P1V0_VCC_FPGA_B"
-		(shape input)
+		(shape output)
 		(at 33.02 35.56 180)
 		(effects
@@
 	)
 	(global_label "P1V0_MGTAVCC_B"
-		(shape input)
+		(shape output)
 		(at 34.29 67.31 180)
 		(effects
@@
 	)
 	(global_label "P1V8_FPGA_VCCAUX_B"
-		(shape input)
+		(shape output)
 		(at 36.83 20.32 180)
 		(effects
@@
 	)
 	(global_label "P1V2_MGTAVTT_B"
-		(shape input)
+		(shape output)
 		(at 34.29 82.55 180)
 		(effects
@@
 	)
 	(global_label "VCC_BANK34_B"
-		(shape output)
+		(shape input)
 		(at 203.2 80.01 0)
 		(effects
@@
 		(on_board yes)
 		(dnp no)
-		(property "Reference" "U1F"
+		(property "Reference" "U1F1"
 			(at 175.26 13.97 0)
 			(effects
@@
 			(project "PicoEVB"
 				(path "/425a64d6-34ec-416c-8211-1f7c9aeb5428/00000000-0000-0000-0000-00005881899d"
-					(reference "U1F")
+					(reference "U1F1")
 					(unit 6)
 				)
@@
 			)
 		)
-		(property "Footprint" "Capacitors_SMD:C_0603"
+		(property "Footprint" "fp_archive:C_0603"
 			(at 136.8552 76.2 0)
 			(effects
@@
 			)
 		)
-		(property "Footprint" "Capacitors_SMD:C_0603"
+		(property "Footprint" "fp_archive:C_0603"
 			(at 136.8552 87.63 0)
 			(effects
@@
 			)
 		)
-		(property "Footprint" "LEDs:LED_0402"
+		(property "Footprint" "fp_archive:LED_0402"
 			(at 128.27 157.48 0)
 			(effects
@@
 			)
 		)
-		(property "Footprint" "Capacitors_SMD:C_0603"
+		(property "Footprint" "fp_archive:C_0603"
 			(at 41.6052 27.94 0)
 			(effects
@@
 			)
 		)
-		(property "Footprint" "Capacitors_SMD:C_0603"
+		(property "Footprint" "fp_archive:C_0603"
 			(at 136.8552 52.07 0)
 			(effects
@@
 		(on_board yes)
 		(dnp no)
-		(property "Reference" "U1A"
+		(property "Reference" "U1A1"
 			(at 115.57 106.68 0)
 			(effects
@@
 			)
 		)
-		(property "Footprint" ""
+		(property "Footprint" "XC7A50T-CSG325:CSG-324"
 			(at 114.3 110.49 0)
 			(effects
@@
 			(project "PicoEVB"
 				(path "/425a64d6-34ec-416c-8211-1f7c9aeb5428/00000000-0000-0000-0000-00005881899d"
-					(reference "U1A")
+					(reference "U1A1")
 					(unit 1)
 				)
@@
 			)
 		)
-		(property "Footprint" "Capacitors_SMD:C_0603"
+		(property "Footprint" "fp_archive:C_0603"
 			(at 136.8552 64.77 0)
 			(effects
@@
 			)
 		)
-		(property "Footprint" "Capacitors_SMD:C_0805"
+		(property "Footprint" "fp_archive:C_0805"
 			(at 40.3352 59.69 0)
 			(effects
@@
 			)
 		)
-		(property "Footprint" "Resistors_SMD:R_Array_Convex_4x0402"
+		(property "Footprint" "Resistor_SMD:R_Array_Convex_4x0402"
 			(at 93.98 151.765 90)
 			(effects
