File: designs/schematics/header_io.kicad_sch (KiCad schematic)
At the start: 2 parts, among them J2 2.54mm Through-Hole Socket, J3 2.54mm Through-Hole Socket

Commit message: Add files via upload
Parts:
- added C70: 0.47uf, SMT:c_0201_least, symbol PicoEVB-rescue:C
- J2, J3: footprint (none) -> Connector_PinHeader_2.54mm:PinHeader_1x39_P2.54mm_Vertical
Connections:
- net GND: now also C70.1
- removed net IO_CONN_3V3: J2.1 (Pin_1), J2.39 (Pin_39), J3.1 (Pin_1), J3.39 (Pin_39)
- new net +3V3: C70.2
