File: designs/schematics/power_b.kicad_sch (KiCad schematic)
At the start: 31 parts, among them J10 1P2, J11 1P0, J12 GND, J7 3P3, J8 1P8, J9 1P0, U3 TPS82085SIL, U4 MAX1589AETT100T, U5 MIC47050-1.2YML, U6 TPS82085SIL

Commit message: Add files via upload
Parts:
- removed C70: 0.47uf, SMT:c_0201_least, symbol PicoEVB-rescue:C
- C53, C54, C55, C57, C62, C63, C65, C66: footprint Capacitors_SMD:C_0805 -> fp_archive:C_0805
- C56, C64: footprint Capacitors_SMD:C_0603 -> fp_archive:C_0603
- J10, J11, J12, J7, J8, J9: footprint Wire_Pads:SolderWirePad_single_SMD_1x1mm -> Connector_Wire:SolderWire-1sqmm_1x01_D1.4mm_OD2.7mm
Other:
- note added: "probing points???"
