File: designs/fpga_io_b.kicad_sch (KiCad schematic)
At the start: 10 parts, among them U1B1 XC7AxxT-xCSG325, U1C1 XC7AxxT-xCSG325, U1D1 XC7AxxT-xCSG325, U2 S25Q

Commit message: Add files via upload
Parts:
- renumbered U1D1 to U1, U1C1 to U1, U1B1 to U1
Changed lines of the file:
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@@
 		(on_board yes)
 		(dnp no)
-		(property "Reference" "U1D1"
+		(property "Reference" "U1"
 			(at 129.54 67.31 0)
 			(effects
@@
 			(project "PicoEVB"
 				(path "/425a64d6-34ec-416c-8211-1f7c9aeb5428/00000000-0000-0000-0000-0000594f323a"
-					(reference "U1D1")
+					(reference "U1")
 					(unit 4)
 				)
@@
 		(on_board yes)
 		(dnp no)
-		(property "Reference" "U1C1"
+		(property "Reference" "U1"
 			(at 69.85 26.67 0)
 			(effects
@@
 			(project "PicoEVB"
 				(path "/425a64d6-34ec-416c-8211-1f7c9aeb5428/00000000-0000-0000-0000-0000594f323a"
-					(reference "U1C1")
+					(reference "U1")
 					(unit 3)
 				)
@@
 		(on_board yes)
 		(dnp no)
-		(property "Reference" "U1B1"
+		(property "Reference" "U1"
 			(at 223.52 26.67 0)
 			(effects
@@
 			(project "PicoEVB"
 				(path "/425a64d6-34ec-416c-8211-1f7c9aeb5428/00000000-0000-0000-0000-0000594f323a"
-					(reference "U1B1")
+					(reference "U1")
 					(unit 2)
 				)
