File: designs/fpga_pcie_b.kicad_sch (KiCad schematic)
At the start: 2 parts, among them U1E1 XC7AxxT-xCSG325

Commit message: Add files via upload
Parts:
- renumbered U1E1 to U1
Changed lines of the file:
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@@
 		(on_board yes)
 		(dnp no)
-		(property "Reference" "U1E1"
+		(property "Reference" "U1"
 			(at 120.65 45.72 0)
 			(effects
@@
 			(project "PicoEVB"
 				(path "/425a64d6-34ec-416c-8211-1f7c9aeb5428/00000000-0000-0000-0000-0000594f3239"
-					(reference "U1E1")
+					(reference "U1")
 					(unit 5)
 				)
