File: designs/M2_edge_b.kicad_sch (KiCad schematic)
At the start: 11 parts, among them J1 Bus_PCI_Express_x4, P2 USB_C_Plug_USB2.0

Commit message: Add files via upload
Connections:
- net +3V3: now also J1.A2 (+12V), J1.A3 (+12V), J1.B1 (+12V), J1.B10 (3.3Vaux), J1.B2 (+12V), J1.B3 (+12V)
- no-connect marks 28 -> 26
