File: designs/fpga_pwr_cfg_b.kicad_sch (KiCad schematic)
At the start: 54 parts, among them U1A1 XC7AxxT-xCSG325, U1F1 XC7AxxT-xCSG325

Commit message: Add files via upload
Parts:
- U1: renamed from U1A1; footprint XC7A50T-CSG325:CSG-324 -> (none); MFG Xilinx -> (none); MPN XC7A50T-2CSG325C -> (none)
- renumbered U1F1 to U1
Changed lines of the file:
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@@
 		(on_board yes)
 		(dnp no)
-		(property "Reference" "U1F1"
+		(property "Reference" "U1"
 			(at 175.26 13.97 0)
 			(effects
@@
 			(project "PicoEVB"
 				(path "/425a64d6-34ec-416c-8211-1f7c9aeb5428/00000000-0000-0000-0000-00005881899d"
-					(reference "U1F1")
+					(reference "U1")
 					(unit 6)
 				)
@@
 		(on_board yes)
 		(dnp no)
-		(property "Reference" "U1A1"
+		(property "Reference" "U1"
 			(at 115.57 106.68 0)
 			(effects
@@
 			)
 		)
-		(property "Footprint" "XC7A50T-CSG325:CSG-324"
+		(property "Footprint" ""
 			(at 114.3 110.49 0)
 			(effects
@@
 			)
 		)
-		(property "MFG" "Xilinx"
-			(at 114.3 110.49 0)
-			(effects
-				(font
-					(size 1.524 1.524)
-				)
-				(hide yes)
-			)
-		)
-		(property "MPN" "XC7A50T-2CSG325C"
-			(at 134.62 151.13 0)
-			(effects
-				(font
-					(size 1.524 1.524)
-				)
-			)
-		)
 		(pin "E1"
 		)
@@
 			(project "PicoEVB"
 				(path "/425a64d6-34ec-416c-8211-1f7c9aeb5428/00000000-0000-0000-0000-00005881899d"
-					(reference "U1A1")
+					(reference "U1")
 					(unit 1)
 				)

Commit message: Add files via upload
Connections:
- net +3V3 renamed VCC_BANK14_B
